File: ES_RearECU_HW.kicad_sch (KiCad schematic)
At the start: 112 parts, among them J1 Conn_02x02_Top_Bottom, J2 Conn_02x02_Top_Bottom, J3 Conn_02x02_Top_Bottom, J4 Conn_02x06_Top_Bottom, J5 Conn_02x04_Top_Bottom, J6 Conn_02x03_Top_Bottom, J7 Conn_02x03_Top_Bottom, K1 FINDER-43.41, K2 FINDER-43.41, K3 FINDER-43.41, Q1 SQ2337CES, Q2 SQ2337CES, Q3 2N7002K, Q4 2N7002K, Q5 2N7002K, Q6 2N7002K, Q7 2N7002K, Q8 2N7002K, SW1 SW_Nidec_CAS-120A1, SW2 SW_Nidec_CAS-120A1, SW3 SW_Push, U1 173010335, U2 173010578, U3 INA186A3, U4 TLV1824, U5 TLV9302xPW, U6 STM32G474CETx, U7 SN65HVD232, U8 TLV9302xPW, Y1 Crystal

Commit message: Canvi mes un conector de prova
Parts:
- added J8: Conn_02x02_Top_Bottom, Connector_Molex:Molex_Nano-Fit_105314-xx04_2x02_P2.50mm_Horizontal, symbol Connector_Generic:Conn_02x02_Top_Bottom
Changed lines of the file:
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@@
+	)
+	(symbol
+		(lib_id "Connector_Generic:Conn_02x02_Top_Bottom")
+		(at 72.39 34.29 0)
+		(unit 1)
+		(exclude_from_sim no)
+		(in_bom yes)
+		(on_board yes)
+		(dnp no)
+		(fields_autoplaced yes)
+		(property "Reference" "J8"
+			(at 73.66 27.94 0)
+			(effects
+				(font
+					(size 1.27 1.27)
+				)
+			)
+		)
+		(property "Value" "Conn_02x02_Top_Bottom"
+			(at 73.66 30.48 0)
+			(effects
+				(font
+					(size 1.27 1.27)
+				)
+			)
+		)
+		(property "Footprint" "Connector_Molex:Molex_Nano-Fit_105314-xx04_2x02_P2.50mm_Horizontal"
+			(at 72.39 34.29 0)
+			(effects
+				(font
+					(size 1.27 1.27)
+				)
+				(hide yes)
+			)
+		)
+		(property "Datasheet" "~"
+			(at 72.39 34.29 0)
+			(effects
+				(font
+					(size 1.27 1.27)
+				)
+				(hide yes)
+			)
+		)
+		(property "Description" "105314"
+			(at 72.39 34.29 0)
+			(effects
+				(font
+					(size 1.27 1.27)
+				)
+				(hide yes)
+			)
+		)
+		(pin "3"
+		)
+		(pin "1"
+		)
+		(pin "2"
+		)
+		(pin "4"
+		)
+		(instances
+			(project "ES_RearECU_HW"
+				(path "/c7bdc31a-c0cb-438d-8083-b4aa911f215a"
+					(reference "J8")
+					(unit 1)
+				)
+			)
+		)
 	)
 	(symbol
